File: kicad/magic-switchboard/_saved_magic-switchboard.sch (KiCad schematic (older format))
At the start: 22 parts, among them Q1 BC547, Q2 BS250, Q3 2N7000, Q4 2N7000, Q5 2N7000, Q6 2N7000, U1 XY-016, U2 alternative Boost Converter

Commit message: created gerbers for v3
Parts:
- U2: value alternative Boost Converter -> 5V Boost Converter
Changed lines of the file:
@@
 P 3400 1400
 F 0 "U2" H 3400 1665 50  0000 C CNN
-F 1 "alternative Boost Converter" H 3400 1574 50  0000 C CNN
+F 1 "5V Boost Converter" H 3400 1574 50  0000 C CNN
 F 2 "switchboard:BoostConverter3Pin" H 3400 1400 50  0001 C CNN
 F 3 "" H 3400 1400 50  0001 C CNN
@@
 	2950 1400 2950 2250
 Wire Wire Line
+	4050 1400 4050 2250
+Wire Wire Line
 	3700 1400 4050 1400
-Wire Wire Line
-	4050 1400 4050 2250
 $EndSCHEMATC
